Commit message: update triangle mesh scale

File: assets/terrains/triangle_mesh/triangle_mesh.urdf (robot description, URDF)
Before this commit: robot triangle_mesh, 1 links, 0 joints
Links:
- link terrainLink: geometry collision mesh filename=terrain9735.obj scale=0.5 0.25 3; visual mesh filename=terrain9735.obj scale=0.5 0.25 3

Commit message: change box terrain

File: assets/terrains/triangle_mesh/triangle_mesh.urdf (robot description, URDF)
Before this commit: robot triangle_mesh, 1 links, 0 joints
Links:
- link terrainLink: geometry collision mesh filename=terrain9735.obj scale=0.5 0.2 2; visual mesh filename=terrain9735.obj scale=0.5 0.2 2
