Commit message: mountain range

File: assets/terrains/mountain_range/mountain_range.urdf (robot description, URDF)
Before this commit: robot triangle_mesh, 1 links, 0 joints
Links:
- removed link terrainLink
- added link mountain_range, mass .0; collision mesh filename=meshes/mountain_range.obj scale=0.01 0.01 0.01; visual mesh filename=meshes/mountain_range.obj scale=0.01 0.01 0.01
