Commit message: fix visual collision mismatch

File: assets/terrains/downladder/downladder.urdf (robot description, URDF)
Before this commit: robot ladder_terrain, 1 links, 0 joints
Links:
- link ladder_terrain: geometry collision mesh filename=meshes/ladder.obj scale=2 0.3 1; visual mesh filename=meshes/ladder.obj scale=2 0.5 1

File: assets/terrains/upladder/upladder.urdf (robot description, URDF)
Before this commit: robot ladder_terrain, 1 links, 0 joints
Links:
- link ladder_terrain: geometry collision mesh filename=meshes/ladder.obj scale=2 0.3 1; visual mesh filename=meshes/ladder.obj scale=2 0.5 1
